File: board/extender/extender.kicad_pcb (KiCad board)
At the start: 2 copper layers, 66 x 53.3 mm, 7 parts, among them J1 EDAC 395-040-559-212, J2 Pin Header, P1 Card Edge

Commit message: Change extender board to 4-layer.
Routing:
- net GND: track 125.2 -> 13.4 mm, vias 0 -> 2
- added copper zone on In1.Cu, net GND
- added copper zone on In2.Cu, net GND
Other:
- copper layers 2 -> 4
